Commit message: 增加关节摩擦，修正urdf中轮子的limit值，第三次训练验证

File: resources/robots/M3/urdf/M3.urdf (robot description, URDF)
Before this commit: robot M3, 17 links, 16 joints
Joints:
- joint FL_foot_joint: limit lower=-3.14 upper=3.14 effort=6.47 velocity=54.873 -> lower=-999999 upper=999999 effort=6.47 velocity=54.873
- joint FR_foot_joint: limit lower=-3.14 upper=3.14 effort=6.47 velocity=54.873 -> lower=-999999 upper=999999 effort=6.47 velocity=54.873
- joint RL_foot_joint: limit lower=-3.14 upper=3.14 effort=6.47 velocity=54.873 -> lower=-999999 upper=999999 effort=6.47 velocity=54.873
- joint RR_foot_joint: limit lower=-3.14 upper=3.14 effort=6.47 velocity=54.873 -> lower=-999999 upper=999999 effort=6.47 velocity=54.873

Commit message: 修正imu坐标

File: resources/robots/M3/urdf/M3.urdf (robot description, URDF)
Before this commit: robot M3, 17 links, 16 joints
Links:
- added link imu, mass 0
Joints:
- added joint imu_joint: type fixed, parent base, child imu, origin xyz=-0.00583 0.00201 0.00949 rpy=0 0 0, axis 0 0 0

Commit message: 修正urdf中髋关节限位和m3.xml中轮子和髋关节限位，第四次训练结果

File: resources/robots/M3/urdf/M3.urdf (robot description, URDF)
Before this commit: robot M3, 18 links, 17 joints
Joints:
- joint FL_hip_joint: limit lower=-0.4 upper=0.4 effort=40 velocity=16.76 -> lower=-1.0 upper=1.0 effort=40 velocity=16.76
- joint FR_hip_joint: limit lower=-0.4 upper=0.4 effort=40 velocity=16.76 -> lower=-1.0 upper=1.0 effort=40 velocity=16.76
- joint RL_hip_joint: limit lower=-0.4 upper=0.4 effort=40 velocity=16.76 -> lower=-1.0 upper=1.0 effort=40 velocity=16.76
- joint RR_hip_joint: limit lower=-0.4 upper=0.4 effort=40 velocity=16.76 -> lower=-1.0 upper=1.0 effort=40 velocity=16.76

Commit message: 调试网络输出中

File: resources/robots/M3/urdf/M3.urdf (robot description, URDF)
Before this commit: robot M3, 18 links, 17 joints
Links:
- link FL_calf: mass 0.33181582 -> 0.77089; geometry collision box size=0.04 0.05 0.162; visual mesh filename=/home/lkz/HIMLoco-for-M3/resources/robots/M3/mjcf/assets/FL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
- link FL_foot: mass 0.64923706 -> 0.254; geometry collision cylinder length=0.035 radius=0.07; visual mesh filename=/home/lkz/HIMLoco-for-M3/resources/robots/M3/mjcf/assets/FL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
- link FL_hip: geometry collision cylinder length=0.06 radius=0.05; visual mesh filename=/home/lkz/HIMLoco-for-M3/resources/robots/M3/mjcf/assets/FL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
- link FL_thigh: mass 1.41948245 -> 1.5045; geometry collision box size=0.090 0.05 0.262; visual mesh filename=/home/lkz/HIMLoco-for-M3/resources/robots/M3/mjcf/assets/FL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
- link FR_calf: mass 0.32996118 -> 0.77089; geometry collision box size=0.04 0.05 0.162; visual mesh filename=/home/lkz/HIMLoco-for-M3/resources/robots/M3/mjcf/assets/FR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
- link FR_foot: mass 0.64923706 -> 0.254; geometry collision cylinder length=0.035 radius=0.07; visual mesh filename=/home/lkz/HIMLoco-for-M3/resources/robots/M3/mjcf/assets/FR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
- link FR_hip: geometry collision cylinder length=0.06 radius=0.05; visual mesh filename=/home/lkz/HIMLoco-for-M3/resources/robots/M3/mjcf/assets/FR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
- link FR_thigh: mass 1.42130584 -> 1.5063; geometry collision box size=0.090 0.05 0.262; visual mesh filename=/home/lkz/HIMLoco-for-M3/resources/robots/M3/mjcf/assets/FR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
- link RL_calf: mass 0.32996118 -> 0.77088638; geometry collision box size=0.04 0.05 0.162; visual mesh filename=/home/lkz/HIMLoco-for-M3/resources/robots/M3/mjcf/assets/RL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
- link RL_foot: mass 0.64923706 -> 0.254; geometry collision cylinder length=0.035 radius=0.07; visual mesh filename=/home/lkz/HIMLoco-for-M3/resources/robots/M3/mjcf/assets/RL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
- link RL_hip: mass 1.04158685 -> 1.0416; geometry collision cylinder length=0.06 radius=0.05; visual mesh filename=/home/lkz/HIMLoco-for-M3/resources/robots/M3/mjcf/assets/RL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
- link RL_thigh: mass 1.41999688 -> 1.50500248; geometry collision box size=0.090 0.05 0.262; visual mesh filename=/home/lkz/HIMLoco-for-M3/resources/robots/M3/mjcf/assets/RL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
- link RR_calf: mass 0.32996118 -> 0.77089; geometry collision box size=0.04 0.05 0.162; visual mesh filename=/home/lkz/HIMLoco-for-M3/resources/robots/M3/mjcf/assets/RR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
- link RR_foot: mass 0.64923706 -> 0.254; geometry collision cylinder length=0.035 radius=0.07; visual mesh filename=/home/lkz/HIMLoco-for-M3/resources/robots/M3/mjcf/assets/RR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
- link RR_hip: mass 1.04158685 -> 1.0416; geometry collision cylinder length=0.06 radius=0.05; visual mesh filename=/home/lkz/HIMLoco-for-M3/resources/robots/M3/mjcf/assets/RR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
- link RR_thigh: mass 1.37914359 -> 1.4641; geometry collision box size=0.090 0.05 0.262; visual mesh filename=/home/lkz/HIMLoco-for-M3/resources/robots/M3/mjcf/assets/RR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
- link base: mass 5.44847063 -> 5.2617; geometry collision box size=0.407 0.240 0.123; visual mesh filename=/home/lkz/HIMLoco-for-M3/resources/robots/M3/mjcf/assets/ba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
Joints:
- joint FL_foot_joint: axis 0 1 0 -> 0 0.99999 0.0033901; origin xyz=0.010478 -0.0155 -0.22676 rpy=0 0 0 -> xyz=0.010478 -0.014013 -0.22635 rpy=0 0 0
- joint FL_hip_joint: limit lower=-1.0 upper=1.0 effort=40 velocity=16.76 -> lower=-0.4 upper=0.4 effort=40 velocity=16.76; origin xyz=0.18927 0.062273 0.059297 rpy=0 0 0 -> xyz=0.18927 0.062072 0.059508 rpy=0 0 0
- joint FR_hip_joint: limit lower=-1.0 upper=1.0 effort=40 velocity=16.76 -> lower=-0.4 upper=0.4 effort=40 velocity=16.76; origin xyz=0.18927 -0.057726 0.059689 rpy=-0.021074 0 0 -> xyz=0.18927 -0.057928 0.059493 rpy=-0.017684 0 0
- joint RL_hip_joint: limit lower=-1.0 upper=1.0 effort=40 velocity=16.76 -> lower=-0.4 upper=0.4 effort=40 velocity=16.76; origin xyz=-0.18913 0.062273 0.059297 rpy=0.045894 0 0 -> xyz=-0.18913 0.062072 0.059508 rpy=0.049284 0 0
- joint RR_hip_joint: limit lower=-1.0 upper=1.0 effort=40 velocity=16.76 -> lower=-0.4 upper=0.4 effort=40 velocity=16.76; origin xyz=-0.18913 -0.057726 0.059689 rpy=-0.021074 0 0 -> xyz=-0.18913 -0.057928 0.059493 rpy=-0.017684 0 0
- joint imu_joint: origin xyz=-0.00583 0.00201 0.00949 rpy=0 0 0 -> xyz=-0.005831 0.001984 0.009498 rpy=0 0 0

Commit message: 调整碰撞以及消除碰撞奖励振荡

File: resources/robots/M3/urdf/M3.urdf (robot description, URDF)
Before this commit: robot M3, 18 links, 17 joints
Links:
- link FL_calf: mass 0.77089 -> 0.7708; geometry collision box size=0.04 0.04 0.152; visual mesh filename=/home/lkz/HIMLoco-for-M3/resources/robots/M3/mjcf/assets/FL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
- link FL_thigh: mass 1.5045 -> 1.5034; geometry collision box size=0.05 0.05 0.12; visual mesh filename=/home/lkz/HIMLoco-for-M3/resources/robots/M3/mjcf/assets/FL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
- link FR_calf: mass 0.77089 -> 0.7708; geometry collision box size=0.04 0.04 0.152; visual mesh filename=/home/lkz/HIMLoco-for-M3/resources/robots/M3/mjcf/assets/FR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
- link FR_thigh: mass 1.5063 -> 1.5034; geometry collision box size=0.05 0.05 0.12; visual mesh filename=/home/lkz/HIMLoco-for-M3/resources/robots/M3/mjcf/assets/FR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
- link RL_calf: mass 0.77088638 -> 0.7708; geometry collision box size=0.04 0.04 0.152; visual mesh filename=/home/lkz/HIMLoco-for-M3/resources/robots/M3/mjcf/assets/RL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
- link RL_thigh: mass 1.50500248 -> 1.5034; geometry collision box size=0.05 0.05 0.112; visual mesh filename=/home/lkz/HIMLoco-for-M3/resources/robots/M3/mjcf/assets/RL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
- link RR_calf: mass 0.77089 -> 0.7708; geometry collision box size=0.04 0.04 0.152; visual mesh filename=/home/lkz/HIMLoco-for-M3/resources/robots/M3/mjcf/assets/RR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
- link RR_thigh: mass 1.4641 -> 1.5034; geometry collision box size=0.05 0.05 0.112; visual mesh filename=/home/lkz/HIMLoco-for-M3/resources/robots/M3/mjcf/assets/RR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
Joints:
- joint FL_hip_joint: limit lower=-0.4 upper=0.4 effort=40 velocity=16.76 -> lower=-1.0472 upper=1.0472 effort=40 velocity=16.76
- joint FR_hip_joint: limit lower=-0.4 upper=0.4 effort=40 velocity=16.76 -> lower=-1.0472 upper=1.0472 effort=40 velocity=16.76
- joint RL_hip_joint: limit lower=-0.4 upper=0.4 effort=40 velocity=16.76 -> lower=-1.0472 upper=1.0472 effort=40 velocity=16.76
- joint RR_hip_joint: limit lower=-0.4 upper=0.4 effort=40 velocity=16.76 -> lower=-1.0472 upper=1.0472 effort=40 velocity=16.76

Commit message: 修正joint axis

File: resources/robots/M3/urdf/M3.urdf (robot description, URDF)
Before this commit: robot M3, 18 links, 17 joints
Joints:
- joint FL_foot_joint: axis 0 0.99999 0.0033901 -> 0 1 0
- joint FR_calf_joint: axis 0 0.99984 0.017805 -> 0 1 0
- joint FR_thigh_joint: axis 0 0.99984 0.017805 -> 0 1 0

Commit message: 修正部分关节参数偏差

File: resources/robots/M3/urdf/M3.urdf (robot description, URDF)
Before this commit: robot M3, 18 links, 17 joints
Joints:
- joint FL_foot_joint: origin xyz=0.010478 -0.014013 -0.22635 rpy=0 0 0 -> xyz=0.010478 -0.014013 -0.221627 rpy=0 0 0
- joint FR_foot_joint: origin xyz=0.0036099 0.024038 -0.22658 rpy=0.017806 0 0 -> xyz=0.0036099 0.024038 -0.220277 rpy=0 0 0
- joint FR_hip_joint: origin xyz=0.18927 -0.057928 0.059493 rpy=-0.017684 0 0 -> xyz=0.18927 -0.057928 0.059493 rpy=0 0 0
- joint RL_foot_joint: origin xyz=0.0034722 -0.02 -0.22697 rpy=0 0 0 -> xyz=0.0034722 -0.02 -0.230432 rpy=0 0 0
- joint RL_hip_joint: origin xyz=-0.18913 0.062072 0.059508 rpy=0.049284 0 0 -> xyz=-0.18913 0.062072 0.059508 rpy=0 0 0
- joint RR_foot_joint: origin xyz=0.0083461 0.02 -0.22685 rpy=0 0 0 -> xyz=0.0083461 0.02 -0.234416 rpy=0 0 0
- joint RR_hip_joint: origin xyz=-0.18913 -0.057928 0.059493 rpy=-0.017684 0 0 -> xyz=-0.18913 -0.057928 0.059493 rpy=0 0 0
