Commit message: 可部署

File: resources/robots/M3/urdf/M3.urdf (robot description, URDF)
Before this commit: robot M3, 18 links, 17 joints
Links:
- link FL_calf: geometry collision box size=0.04 0.03 0.132; visual mesh filename=/home/lkz/HIMLoco-for-M3/resources/robots/M3/mjcf/assets/FL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
- link FR_calf: geometry collision box size=0.04 0.03 0.132; visual mesh filename=/home/lkz/HIMLoco-for-M3/resources/robots/M3/mjcf/assets/FR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
- link RL_calf: geometry collision box size=0.04 0.03 0.132; visual mesh filename=/home/lkz/HIMLoco-for-M3/resources/robots/M3/mjcf/assets/RL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
- link RR_calf: geometry collision box size=0.04 0.03 0.132; visual mesh filename=/home/lkz/HIMLoco-for-M3/resources/robots/M3/mjcf/assets/RR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
Joints:
- joint FL_foot_joint: limit lower=-999999 upper=999999 effort=6.47 velocity=54.873 -> lower=-999999 upper=999999 effort=6.47 velocity=27.873; origin xyz=0.010478 -0.014013 -0.221627 rpy=0 0 0 -> xyz=0.010478 -0.014013 -0.224907609 rpy=0 0 0
- joint FR_foot_joint: limit lower=-999999 upper=999999 effort=6.47 velocity=54.873 -> lower=-999999 upper=999999 effort=6.47 velocity=27.873; origin xyz=0.0036099 0.024038 -0.220277 rpy=0 0 0 -> xyz=0.0036099 0.024038 -0.221027458 rpy=0 0 0
- joint RL_foot_joint: limit lower=-999999 upper=999999 effort=6.47 velocity=54.873 -> lower=-999999 upper=999999 effort=6.47 velocity=27.873; origin xyz=0.0034722 -0.02 -0.230432 rpy=0 0 0 -> xyz=0.0034722 -0.02 -0.225832115 rpy=0 0 0
- joint RR_foot_joint: limit lower=-999999 upper=999999 effort=6.47 velocity=54.873 -> lower=-999999 upper=999999 effort=6.47 velocity=27.873; origin xyz=0.0083461 0.02 -0.234416 rpy=0 0 0 -> xyz=0.0083461 0.02 -0.234984818 rpy=0 0 0
